Commit message: working...

File: src/testbot_description/urdf/physical_properties.xacro (robot description, xacro)
@@ -2,6 +2,6 @@
 <robot xmlns:xacro="http://www.ros.org/wiki/xacro">
     <!-- Robot Dimensions -->
-    <xacro:property name="robot_length" value="0.18"/>  <!-- 18 cm -->
-    <xacro:property name="robot_width" value="0.12"/>   <!-- 12 cm -->
+    <xacro:property name="robot_length" value="0.18"/>      <!-- 18 cm -->
+    <xacro:property name="robot_width" value="0.12"/>       <!-- 12 cm -->
     <xacro:property name="wheel_separation" value="0.13"/>  <!-- 13 cm -->
     <xacro:property name="wheel_radius" value="0.022"/>     <!-- 44mm diameter -->

File: src/testbot_description/urdf/testbot.urdf.xacro (robot description, xacro)
@@ -1,7 +1,5 @@
 <?xml version="1.0"?>
 <robot name="testbot" xmlns:xacro="http://www.ros.org/wiki/xacro">
-  <!-- Include Physical Properties -->
   <xacro:include filename="$(find testbot_description)/urdf/physical_properties.xacro"/>
-  <!-- Materials -->
   <material name="black">
     <color rgba="0.0 0.0 0.0 1.0"/>
@@ -10,5 +8,4 @@
     <color rgba="0.0 0.0 0.8 1.0"/>
   </material>
-  <!-- Base Link -->
   <link name="base_footprint"/>
   <joint name="base_joint" type="fixed">
@@ -38,5 +35,4 @@
     </inertial>
   </link>
-  <!-- Left Wheel -->
   <joint name="left_wheel_joint" type="continuous">
     <parent link="base_link"/>
@@ -64,5 +60,4 @@
     </inertial>
   </link>
-  <!-- Right Wheel -->
   <joint name="right_wheel_joint" type="continuous">
     <parent link="base_link"/>
@@ -90,5 +85,4 @@
     </inertial>
   </link>
-  <!-- Caster Wheel -->
   <joint name="caster_joint" type="fixed">
     <parent link="base_link"/>
