Commit message: udpate slam config

File: src/testbot_description/urdf/testbot.urdf.xacro (robot description, xacro)
@@ -109,3 +109,28 @@
     </inertial>
   </link>
+  <joint name="laser_joint" type="fixed">
+    <parent link="base_link"/>
+    <child link="laser"/>
+    <origin xyz="0.0 0.0 0.08" rpy="0 0 0"/>  <!-- Adjust XYZ based on actual position -->
+  </joint>
+  <!-- RPLidar link -->
+  <link name="laser">
+    <visual>
+      <geometry>
+        <cylinder length="0.04" radius="0.025"/>
+      </geometry>
+      <material name="black"/>
+    </visual>
+    <collision>
+      <geometry>
+        <cylinder length="0.04" radius="0.025"/>
+      </geometry>
+    </collision>
+    <inertial>
+      <mass value="0.1"/>
+      <inertia ixx="0.001" ixy="0.0" ixz="0.0"
+               iyy="0.001" iyz="0.0"
+               izz="0.001"/>
+    </inertial>
+  </link>
 </robot>
